Commit message: [New Robot] 添加Taks_T1机器人支持，包含ground、platform、wall、slope和ground_prone五种环境配置，并在URDF中新增关键帧链接

File: legged_gym/resources/robots/Taks_T1/Taks_T1.urdf (robot description, URDF)
Before this commit: robot Taks_T1, 42 links, 41 joints
Links:
- added link keyframe_head_link
- added link keyframe_left_ankle_link
- added link keyframe_left_collar_link
- added link keyframe_left_elbow_link
- added link keyframe_left_hip_link
- added link keyframe_left_knee_link
- added link keyframe_left_shoulder_link
- added link keyframe_left_wrist_link
- added link keyframe_pelvis_link
- added link keyframe_right_ankle_link
- added link keyframe_right_collar_link
- added link keyframe_right_elbow_link
- added link keyframe_right_hip_link
- added link keyframe_right_knee_link
- added link keyframe_right_shoulder_link
- added link keyframe_right_wrist_link
- added link keyframe_torso_link
Joints:
- added joint keyframe_head_joint: type fixed, parent torso_link, child keyframe_head_link, origin xyz=0 0 0.45 rpy=0 0 0
- added joint keyframe_left_ankle_joint: type fixed, parent left_ankle_roll_link, child keyframe_left_ankle_link, origin xyz=0 0 0 rpy=0 0 0
- added joint keyframe_left_collar_joint: type fixed, parent left_shoulder_pitch_link, child keyframe_left_collar_link, origin xyz=0 0 0.02 rpy=0 0 0
- added joint keyframe_left_elbow_joint: type fixed, parent left_elbow_link, child keyframe_left_elbow_link, origin xyz=0 0 0 rpy=0 0 0
- added joint keyframe_left_hip_joint: type fixed, parent left_hip_roll_link, child keyframe_left_hip_link, origin xyz=0 0 0 rpy=0 0 0
- added joint keyframe_left_knee_joint: type fixed, parent left_knee_link, child keyframe_left_knee_link, origin xyz=0 0 0 rpy=0 0 0
- added joint keyframe_left_shoulder_joint: type fixed, parent left_shoulder_roll_link, child keyframe_left_shoulder_link, origin xyz=0 0 0 rpy=0 0 0
- added joint keyframe_left_wrist_joint: type fixed, parent left_wrist_pitch_link, child keyframe_left_wrist_link, origin xyz=0 0 0 rpy=0 0 0
- added joint keyframe_pelvis_joint: type fixed, parent pelvis, child keyframe_pelvis_link, origin xyz=0 0 -0.075 rpy=0 0 0
- added joint keyframe_right_ankle_joint: type fixed, parent right_ankle_roll_link, child keyframe_right_ankle_link, origin xyz=0 0 0 rpy=0 0 0
- added joint keyframe_right_collar_joint: type fixed, parent right_shoulder_pitch_link, child keyframe_right_collar_link, origin xyz=0 0 0.02 rpy=0 0 0
- added joint keyframe_right_elbow_joint: type fixed, parent right_elbow_link, child keyframe_right_elbow_link, origin xyz=0 0 0 rpy=0 0 0
- added joint keyframe_right_hip_joint: type fixed, parent right_hip_roll_link, child keyframe_right_hip_link, origin xyz=0 0 0 rpy=0 0 0
- added joint keyframe_right_knee_joint: type fixed, parent right_knee_link, child keyframe_right_knee_link, origin xyz=0 0 0 rpy=0 0 0
- added joint keyframe_right_shoulder_joint: type fixed, parent right_shoulder_roll_link, child keyframe_right_shoulder_link, origin xyz=0 0 0 rpy=0 0 0
- added joint keyframe_right_wrist_joint: type fixed, parent right_wrist_pitch_link, child keyframe_right_wrist_link, origin xyz=0 0 0 rpy=0 0 0
- added joint keyframe_torso_joint: type fixed, parent torso_link, child keyframe_torso_link, origin xyz=0 0 0.2 rpy=0 0 0

Commit message: 调整Taks_T1机器人PD控制刚度参数，增加wandb日志支持，修复URDF格式

File: legged_gym/resources/robots/Taks_T1/Taks_T1.urdf (robot description, URDF)
Before this commit: robot Taks_T1, 59 links, 58 joints
Links:
- removed link world
Joints:
- removed joint pelvis
